File: Shield-Attiny/Shield-Attiny.kicad_pcb (KiCad board)
At the start: 2 copper layers, 70.7 x 53.6 mm, 9 parts, among them SW1 SW_Push, U1 ATtiny85-20PU

Commit message: added images and edge cuts
Other:
- board size 70.7 x 53.6 mm -> 75.1 x 53.6 mm
Changed lines of the file:
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@@
   (general
     (thickness 1.6)
-    (drawings 14)
+    (drawings 19)
     (tracks 60)
     (zones 0)
@@
     (35 F.Paste user)
     (36 B.SilkS user)
-    (37 F.SilkS user)
+    (37 F.SilkS user hide)
     (38 B.Mask user)
     (39 F.Mask user)
@@
     (47 F.CrtYd user)
     (48 B.Fab user)
-    (49 F.Fab user)
+    (49 F.Fab user hide)
   )
   (setup
@@
     )
   )
-  (gr_line (start 123.1392 86.9442) (end 123.063 45.6184) (layer Edge.Cuts) (width 0.05))
+  (gr_line (start 123.0884 55.1688) (end 123.063 45.6184) (layer Edge.Cuts) (width 0.05))
+  (gr_line (start 116.7892 55.1688) (end 123.0884 55.1688) (layer Edge.Cuts) (width 0.05))
+  (gr_line (start 116.7892 66.7512) (end 116.7892 55.1688) (layer Edge.Cuts) (width 0.05))
+  (gr_line (start 123.1138 66.7512) (end 116.7892 66.7512) (layer Edge.Cuts) (width 0.05))
+  (gr_line (start 123.1392 86.9442) (end 123.1138 66.7512) (layer Edge.Cuts) (width 0.05))
+  (dimension 66.170128 (width 0.15) (layer Dwgs.User)
+    (gr_text "66.170 mm" (at 156.246519 113.621618 359.8874348) (layer Dwgs.User)
+      (effects (font (size 1 1) (thickness 0.15)))
+    )
+    (feature1 (pts (xy 189.36 99.19) (xy 189.332921 112.97304)))
+    (feature2 (pts (xy 123.19 99.06) (xy 123.162921 112.84304)))
+    (crossbar (pts (xy 123.164073 112.256621) (xy 189.334073 112.386621)))
+    (arrow1a (pts (xy 189.334073 112.386621) (xy 188.206419 112.970827)))
+    (arrow1b (pts (xy 189.334073 112.386621) (xy 188.208724 111.797988)))
+    (arrow2a (pts (xy 123.164073 112.256621) (xy 124.289422 112.845254)))
+    (arrow2b (pts (xy 123.164073 112.256621) (xy 124.291727 111.672415)))
+  )
   (gr_line (start 121.2088 86.9442) (end 123.1392 86.9442) (layer Edge.Cuts) (width 0.05))
   (gr_line (start 121.1834 95.9866) (end 121.2088 86.9442) (layer Edge.Cuts) (width 0.05))
